File: PCB/Hybrid-Pico.kicad_pcb (KiCad board)
At the start: 2 copper layers, 21 x 51 mm, 39 parts, among them J1 USB_C_Receptacle_USB2.0_16P, J2 Conn_01x20, J3 Conn_01x20, J4 Conn_01x03, SW1 SW_Push, U1 RP2040, U2 MCP1700x-330xxTT, U4 W25Q16JVUXIQ TR, U5 MPU-6050, U6 BMP280, Y1 12 MHz

Commit message: Add files via upload
Parts:
- removed R1, R2: 33 R, Capacitor_SMD:C_0201_0603Metric
- added C226: 100 nf, Capacitor_SMD:C_0402_1005Metric, F.Cu at (164.7, 78.3)
- added C232: 100 nf, Capacitor_SMD:C_0201_0603Metric, F.Cu at (172.7, 78.3)
- added C71: 1uF, Capacitor_SMD:C_0402_1005Metric, F.Cu at (175.1, 76.5)
- added C88: 100 nf, Capacitor_SMD:C_0402_1005Metric, F.Cu at (169.6, 88.0)
- added C91: 1uf, Capacitor_SMD:C_0201_0603Metric, F.Cu at (172.0, 78.3)
- added R10: 4.7K, Capacitor_SMD:C_0402_1005Metric, F.Cu at (163.5, 92.6)
- added R104: 4.7K, Capacitor_SMD:C_0402_1005Metric, F.Cu at (173.4, 86.9)
- added R14: 10K, Resistor_SMD:R_0603_1608Metric, F.Cu at (175.4, 71.9)
- added R145: 4.7K, Capacitor_SMD:C_0402_1005Metric, F.Cu at (174.8, 86.9)
- added R15: 4.7K, Capacitor_SMD:C_0402_1005Metric, F.Cu at (165.0, 94.6)
- added R81: 27, Capacitor_SMD:C_0402_1005Metric, F.Cu at (169.9, 77.2)
- added R91: 27, Capacitor_SMD:C_0402_1005Metric, F.Cu at (170.9, 77.2)
- added SW3: SW_Push, Button_Switch_SMD:SW_Push_SPST_NO_Alps_SKRK, F.Cu at (173.9, 68.7)
Connections:
- J3 pad 5: +3V3 -> 3.3V
Routing:
- net 3.3V: track 74.7 -> 114.9 mm, vias 7 -> 15
- net RUN: track 8.85 -> 32.7 mm, vias 1 -> 4
- net GND: track 98.9 -> 114.0 mm, vias 15 -> 20
- net Net-(U1-VREG_VOUT): track 13.4 -> 25.8 mm, vias 2 -> 4
- net _D+: track 13.7 -> 2.11 mm
- net _D-: track 13.7 -> 2.36 mm
- net Net-(J1-D--PadA7): track 4.41 -> 14.5 mm
- net Net-(J1-D+-PadA6): track 4.48 -> 14.3 mm
- net GPIO28_ADC2: track 17.7 -> 18.7 mm
- net GPIO21: track 11.7 -> 12.3 mm
- net GPIO27_ADC1: track 12.9 -> 12.3 mm

Commit message: Add files via upload
Routing:
- net GND: track 114.0 -> 117.7 mm
Changed lines of the file:
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@@
+	)
+	(segment
+		(start 172.354998 88.44)
+		(end 172.354998 91.124998)
+		(width 0.15)
+		(layer "B.Cu")
+		(net 1)
 	)
 	(segment
@@
 		(width 0.15)
 		(layer "B.Cu")
+		(net 1)
+	)
+	(segment
+		(start 172.354998 91.124998)
+		(end 173.08 91.85)
+		(width 0.15)
+		(layer "B.Cu")

Commit message: Add files via upload
Parts:
- R10, R104, R145, R15: value 4.7K -> 5.1K
Connections:
- C71 pad 2: Net-(U1-VREG_VOUT) -> Net-(U10-VREG_VOUT)
- R10 pad 2: 3.3V -> +3.3V
- R15 pad 2: 3.3V -> +3.3V
Changed lines of the file:
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@@
 	(net 78 "Net-(U10-USB_DP)")
 	(net 79 "Net-(U10-USB_DM)")
+	(net 80 "+3.3V")
+	(net 81 "Net-(U10-VREG_VOUT)")
 	(footprint "Capacitor_SMD:C_0402_1005Metric"
 		(layer "F.Cu")
@@
 			(layers "F.Cu" "F.Mask" "F.Paste")
 			(roundrect_rratio 0.25)
-			(net 58 "Net-(U1-VREG_VOUT)")
+			(net 81 "Net-(U10-VREG_VOUT)")
 			(pintype "passive")
 		)
@@
 			)
 		)
-		(property "Value" "4.7K"
+		(property "Value" "5.1K"
 			(at -0.39 0.95 120)
 			(layer "F.Fab")
@@
 			)
 		)
-		(property "Value" "4.7K"
+		(property "Value" "5.1K"
 			(at 0 1.16 90)
 			(layer "F.Fab")
@@
 			(layers "F.Cu" "F.Mask" "F.Paste")
 			(roundrect_rratio 0.25)
-			(net 2 "3.3V")
+			(net 80 "+3.3V")
 			(pintype "passive")
 		)
@@
 			)
 		)
-		(property "Value" "4.7K"
+		(property "Value" "5.1K"
 			(at 0 1.16 90)
 			(layer "F.Fab")
@@
 			)
 		)
-		(property "Value" "4.7K"
+		(property "Value" "5.1K"
 			(at 0 1.16 90)
 			(layer "F.Fab")
@@
 			(layers "F.Cu" "F.Mask" "F.Paste")
 			(roundrect_rratio 0.25)
-			(net 2 "3.3V")
+			(net 80 "+3.3V")
 			(pintype "passive")
 		)
